File: ArcJoy_Pcb/ArcJoy.kicad_pcb (KiCad board)
At the start: 2 copper layers, 95 x 60 mm, 38 parts, among them J1 Conn_01x06, J10 Conn_01x02, J11 Conn_01x02, J12 Conn_01x02, J2 Conn_01x02, J3 Conn_01x02, J4 Conn_01x02, J5 Conn_01x02, J6 Conn_01x02, J7 Conn_01x02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

Commit message: COnversion started
Parts:
- R11: value 10k -> 5k1_1206_1%
- R12: value 10k -> 330R_1206_1%
Connections:
- J10 pad 1: /BUTTON5 -> /BUTTON2
- J11 pad 1: /BUTTON6 -> /BUTTON1
- J6 pad 1: /BUTTON1 -> /BUTTON6
- J7 pad 1: /BUTTON2 -> /BUTTON5
- J8 pad 1: /BUTTON3 -> /BUTTON4
- J9 pad 1: /BUTTON4 -> /BUTTON3
- R1 pad 2: /BUTTON4 -> /BUTTON3
- R10 pad 2: /BUTTON5 -> /BUTTON2
- R2 pad 2: /BUTTON1 -> /BUTTON6
- R3 pad 2: /BUTTON2 -> /BUTTON5
- R4 pad 2: /BUTTON3 -> /BUTTON4
- R6 pad 2: /BUTTON6 -> /BUTTON1
- U1 pad P$21: /BUTTON1 -> /BUTTON6
- U1 pad P$22: /BUTTON2 -> /BUTTON5
- U1 pad P$23: /BUTTON3 -> /BUTTON4
- U1 pad P$24: /BUTTON4 -> /BUTTON3
- U1 pad P$25: /BUTTON5 -> /BUTTON2
- U1 pad P$26: /BUTTON6 -> /BUTTON1
Routing:
- net /BUTTON6: track 52.1 -> 55.3 mm
- net /BUTTON1: track 55.3 -> 52.1 mm
- net /BUTTON5: track 53.9 -> 56.1 mm
- net /BUTTON2: track 56.1 -> 53.9 mm
