File: ArcJoy_Pcb/ArcJoy.kicad_pcb (KiCad board)
At the start: 2 copper layers, 95 x 60 mm, 38 parts, among them J1 Conn_01x06, J10 Conn_01x02, J11 Conn_01x02, J12 Conn_01x02, J2 Conn_01x02, J3 Conn_01x02, J4 Conn_01x02, J5 Conn_01x02, J6 Conn_01x02, J7 Conn_01x02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

Commit message: BOM
Parts:
- R11: value 10k -> 5k1_1206_1%
- R12: value 10k -> 330R_1206_1%
- U2: value MCP1711T-22I_OT -> MCP1711T-25I_OT
Changed lines of the file:
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@@
       (effects (font (size 1 1) (thickness 0.15)))
     )
-    (fp_text value 10k (at 0 1.82 180) (layer F.Fab)
+    (fp_text value 330R_1206_1% (at 0 1.82 180) (layer F.Fab)
       (effects (font (size 1 1) (thickness 0.15)))
     )
@@
       (effects (font (size 1 1) (thickness 0.15)))
     )
-    (fp_text value 10k (at 0 1.82 180) (layer F.Fab)
+    (fp_text value 5k1_1206_1% (at 0 1.82 180) (layer F.Fab)
       (effects (font (size 1 1) (thickness 0.15)))
     )
@@
       (effects (font (size 1 1) (thickness 0.15)))
     )
-    (fp_text value MCP1711T-22I_OT (at 0 2.9 90) (layer F.Fab)
-      (effects (font (size 1 1) (thickness 0.15)))
-    )
+    (fp_text value MCP1711T-25I_OT (at 0 2.9 90) (layer F.Fab)
+      (effects (font (size 1 1) (thickness 0.15)))
+    )
