File: ArcJoy_Pcb/ArcJoy.kicad_pcb (KiCad board)
At the start: 2 copper layers, 95 x 60 mm, 38 parts, among them J1 Conn_01x06, J10 Conn_01x02, J11 Conn_01x02, J12 Conn_01x02, J2 Conn_01x02, J3 Conn_01x02, J4 Conn_01x02, J5 Conn_01x02, J6 Conn_01x02, J7 Conn_01x02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

Commit message: Net +2V2 changed to +2V5
Connections:
- net +2V2 renamed +2V5
