File: ArcJoy_Pcb/ArcJoy.sch (KiCad schematic (older format))
At the start: 35 parts, among them J1 Conn_01x06, J10 Conn_01x02, J11 Conn_01x02, J12 Conn_01x02, J2 Conn_01x02, J3 Conn_01x02, J4 Conn_01x02, J5 Conn_01x02, J6 Conn_01x02, J7 Conn_01x02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

Commit message: COnversion started
Changed lines of the file:
@@
 	1    0    0    -1
 $EndComp
-Text Label 1400 3350 0    50   ~ 0
+Text Label 1400 7100 0    50   ~ 0
 BUTTON1
 $Comp
@@
 	1    0    0    -1
 $EndComp
+Text Label 1400 6350 0    50   ~ 0
+BUTTON2
+Text Label 1400 5600 0    50   ~ 0
+BUTTON3
+Text Label 1400 4850 0    50   ~ 0
+BUTTON4
 Text Label 1400 4100 0    50   ~ 0
+BUTTON5
+Text Label 1400 3350 0    50   ~ 0
+BUTTON6
+Text Label 8950 4800 1    50   ~ 0
+BUTTON1
+Text Label 8850 4800 1    50   ~ 0
 BUTTON2
-Text Label 1400 4850 0    50   ~ 0
-BUTTON3
-Text Label 1400 5600 0    50   ~ 0
-BUTTON4
-Text Label 1400 6350 0    50   ~ 0
-BUTTON5
-Text Label 1400 7100 0    50   ~ 0
-BUTTON6
-Text Label 8450 4800 1    50   ~ 0
-BUTTON1
-Text Label 8550 4800 1    50   ~ 0
-BUTTON2
-Text Label 8650 4800 1    50   ~ 0
+Text Label 8750 4800 1    50   ~ 0
 BUTTON3
 Text Label 8350 4800 1    50   ~ 0
@@
 Wire Wire Line
 	8850 4400 8850 4800
-Text Label 8750 4800 1    50   ~ 0
+Text Label 8650 4800 1    50   ~ 0
 BUTTON4
-Text Label 8850 4800 1    50   ~ 0
+Text Label 8550 4800 1    50   ~ 0
 BUTTON5
-Text Label 8950 4800 1    50   ~ 0
+Text Label 8450 4800 1    50   ~ 0
 BUTTON6
 Wire Wire Line
