File: ArcJoy_Pcb/ArcJoy.sch (KiCad schematic (older format))
At the start: 35 parts, among them J1 Conn_01x06, J10 Conn_01x02, J11 Conn_01x02, J12 Conn_01x02, J2 Conn_01x02, J3 Conn_01x02, J4 Conn_01x02, J5 Conn_01x02, J6 Conn_01x02, J7 Conn_01x02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

Commit message: LEDs and dipswitch managing.
Parts:
- R11: value 10k -> 5k1_1206_1%; symbol K_Resistors:10k_1206_1% -> K_Resistors:5k1_1206_1%; ElementValue (none) -> 5k1; Supplier Part Number 1 1206S4F1002T5E -> SMD1206-5K1-1%
- R12: value 10k -> 330R_1206_1%; symbol K_Resistors:10k_1206_1% -> K_Resistors:330R_1206_1%; ElementValue (none) -> 330R; Supplier Part Number 1 1206S4F1002T5E -> SMD1206-330R-1%
Changed lines of the file:
@@
 LED_B
 $Comp
-L K_Resistors:10k_1206_1% R11
+L K_Resistors:5k1_1206_1% R11
 U 1 1 5CC86B26
 P 4600 6150
-F 0 "R11" V 4700 6000 50  0000 L CNN
-F 1 "10k" V 4500 6150 50  0000 L CNN
+F 0 "R11" V 4500 5900 50  0000 L CNN
+F 1 "5k1_1206_1%" V 4500 6150 50  0001 L CNN
 F 2 "Resistor_SMD:R_1206_3216Metric" H 4600 5400 50  0001 L CNN
 F 3 "~" V 4680 6150 50  0001 C CNN
 F 4 "TME" H 4600 5600 50  0001 L CNN "Supplier 1"
-F 5 "1206S4F1002T5E" H 4600 5500 50  0001 L CNN "Supplier Part Number 1"
+F 5 "SMD1206-5K1-1%" H 4600 5500 50  0001 L CNN "Supplier Part Number 1"
+F 6 "5k1" V 4500 6150 50  0000 C CNN "ElementValue"
 	1    4600 6150
 	0    1    1    0
 $EndComp
 $Comp
-L K_Resistors:10k_1206_1% R12
+L K_Resistors:330R_1206_1% R12
 U 1 1 5CC87CC7
 P 4600 6350
-F 0 "R12" V 4300 6200 50  0000 L CNN
-F 1 "10k" V 4500 6350 50  0000 L CNN
+F 0 "R12" V 4500 6100 50  0000 L CNN
+F 1 "330R_1206_1%" V 4500 6350 50  0001 L CNN
 F 2 "Resistor_SMD:R_1206_3216Metric" H 4600 5600 50  0001 L CNN
 F 3 "~" V 4680 6350 50  0001 C CNN
 F 4 "TME" H 4600 5800 50  0001 L CNN "Supplier 1"
-F 5 "1206S4F1002T5E" H 4600 5700 50  0001 L CNN "Supplier Part Number 1"
+F 5 "SMD1206-330R-1%" H 4600 5700 50  0001 L CNN "Supplier Part Number 1"
+F 6 "330R" V 4500 6350 50  0000 C CNN "ElementValue"
 	1    4600 6350
 	0    1    1    0

Commit message: BOM
Parts:
- U2: value MCP1711T-22I_OT -> MCP1711T-25I_OT; symbol K_Regulators:MCP1711T-22I_OT -> K_Regulators:MCP1711T-25I_OT
Changed lines of the file:
@@
 Napięcie - zmienić na 3V?rewrwe\n
 $Comp
-L K_Regulators:MCP1711T-22I_OT U2
+L K_Regulators:MCP1711T-25I_OT U2
 U 1 1 5CC244C8
 P 5350 4550
 F 0 "U2" H 5350 4892 50  0000 C CNN
-F 1 "MCP1711T-22I_OT" H 5350 4801 50  0000 C CNN
+F 1 "MCP1711T-25I_OT" H 5350 4801 50  0000 C CNN
 F 2 "Package_TO_SOT_SMD:SOT-23-5" H 5350 4900 50  0001 C CNN
 F 3 "ww1.microchip.com/downloads/en/devicedoc/20005415d.pdf" H 5350 4800 50  0001 C CNN

Commit message: Net +2V2 changed to +2V5
Connections:
- net labels added: +2V5
- net labels removed: +2V2
Other:
- note removed: "Napięcie - zmienić na 3V?rewrwe\n"
Changed lines of the file:
@@
 	1    0    0    -1
 $EndComp
-Text Notes 550  950  0    50   ~ 0
-Napięcie - zmienić na 3V?rewrwe\n
 $Comp
 L K_Regulators:MCP1711T-25I_OT U2
@@
 	5950 4450 5950 4350
 $Comp
-L K_Power:+2V2 #PWR0103
-U 1 1 5CC2A9EF
-P 8300 5700
-F 0 "#PWR0103" H 8550 5850 50  0001 C CNN
-F 1 "+2V2" H 8305 5873 50  0000 C CNN
-F 2 "" H 8100 6000 50  0001 C CNN
-F 3 "" H 8100 6000 50  0001 C CNN
-	1    8300 5700
-	1    0    0    -1
-$EndComp
-$Comp
 L power:GND #PWR0104
 U 1 1 5CC318D4
@@
 Wire Wire Line
 	9600 5850 10000 5850
-$Comp
-L K_Power:+2V2 #PWR0108
-U 1 1 5CC3F27E
-P 9300 5350
-F 0 "#PWR0108" H 9550 5500 50  0001 C CNN
-F 1 "+2V2" H 9305 5523 50  0000 C CNN
-F 2 "" H 9100 5650 50  0001 C CNN
-F 3 "" H 9100 5650 50  0001 C CNN
-	1    9300 5350
-	1    0    0    -1
-$EndComp
 Text Label 9650 5450 0    50   ~ 0
 SWCLK
@@
 $EndComp
 $Comp
-L K_Power:+2V2 #PWR0115
-U 1 1 5CC6330B
-P 2250 1550
-F 0 "#PWR0115" H 2500 1700 50  0001 C CNN
-F 1 "+2V2" H 2255 1723 50  0000 C CNN
-F 2 "" H 2050 1850 50  0001 C CNN
-F 3 "" H 2050 1850 50  0001 C CNN
-	1    2250 1550
-	1    0    0    -1
-$EndComp
-$Comp
-L K_Power:+2V2 #PWR0116
-U 1 1 5CC63D9D
-P 3400 900
-F 0 "#PWR0116" H 3650 1050 50  0001 C CNN
-F 1 "+2V2" H 3405 1073 50  0000 C CNN
-F 2 "" H 3200 1200 50  0001 C CNN
-F 3 "" H 3200 1200 50  0001 C CNN
-	1    3400 900
-	1    0    0    -1
-$EndComp
-$Comp
-L K_Power:+2V2 #PWR0117
-U 1 1 5CC642B6
-P 4550 1550
-F 0 "#PWR0117" H 4800 1700 50  0001 C CNN
-F 1 "+2V2" H 4555 1723 50  0000 C CNN
-F 2 "" H 4350 1850 50  0001 C CNN
-F 3 "" H 4350 1850 50  0001 C CNN
-	1    4550 1550
-	1    0    0    -1
-$EndComp
-$Comp
-L K_Power:+2V2 #PWR0118
+L K_Power:+2V5 #PWR0118
 U 1 1 5CC64791
 P 3400 2000
 F 0 "#PWR0118" H 3650 2150 50  0001 C CNN
-F 1 "+2V2" H 3405 2173 50  0000 C CNN
+F 1 "+2V5" H 3405 2173 50  0000 C CNN
 F 2 "" H 3200 2300 50  0001 C CNN
 F 3 "" H 3200 2300 50  0001 C CNN
@@
 $EndComp
 $Comp
-L K_Power:+2V2 #PWR0124
-U 1 1 5CC69306
-P 1800 3050
-F 0 "#PWR0124" H 2050 3200 50  0001 C CNN
-F 1 "+2V2" H 1805 3223 50  0000 C CNN
-F 2 "" H 1600 3350 50  0001 C CNN
-F 3 "" H 1600 3350 50  0001 C CNN
-	1    1800 3050
-	1    0    0    -1
-$EndComp
-$Comp
 L K_Resistors:10k_1206_1% R3
 U 1 1 5CC6ACC6
@@
 $EndComp
 $Comp
-L K_Power:+2V2 #PWR0125
-U 1 1 5CC6ACCE
-P 1800 3800
-F 0 "#PWR0125" H 2050 3950 50  0001 C CNN
-F 1 "+2V2" H 1805 3973 50  0000 C CNN
-F 2 "" H 1600 4100 50  0001 C CNN
-F 3 "" H 1600 4100 50  0001 C CNN
-	1    1800 3800
-	1    0    0    -1
-$EndComp
-$Comp
 L K_Resistors:10k_1206_1% R4
 U 1 1 5CC6C39A
@@
 $EndComp
 $Comp
-L K_Power:+2V2 #PWR0126
-U 1 1 5CC6C3A2
-P 1800 4550
-F 0 "#PWR0126" H 2050 4700 50  0001 C CNN
-F 1 "+2V2" H 1805 4723 50  0000 C CNN
-F 2 "" H 1600 4850 50  0001 C CNN
-F 3 "" H 1600 4850 50  0001 C CNN
-	1    1800 4550
-	1    0    0    -1
-$EndComp
-$Comp
 L K_Resistors:10k_1206_1% R1
 U 1 1 5CC6DEAF
@@
 $EndComp
 $Comp
-L K_Power:+2V2 #PWR0127
-U 1 1 5CC6DEB7
-P 1800 5300
-F 0 "#PWR0127" H 2050 5450 50  0001 C CNN
-F 1 "+2V2" H 1805 5473 50  0000 C CNN
-F 2 "" H 1600 5600 50  0001 C CNN
-F 3 "" H 1600 5600 50  0001 C CNN
-	1    1800 5300
-	1    0    0    -1
-$EndComp
-$Comp
 L K_Resistors:10k_1206_1% R6
 U 1 1 5CC71A05
@@
 $EndComp
 $Comp
-L K_Power:+2V2 #PWR0128
-U 1 1 5CC71A0D
-P 1800 6800
-F 0 "#PWR0128" H 2050 6950 50  0001 C CNN
-F 1 "+2V2" H 1805 6973 50  0000 C CNN
-F 2 "" H 1600 7100 50  0001 C CNN
-F 3 "" H 1600 7100 50  0001 C CNN
-	1    1800 6800
-	1    0    0    -1
-$EndComp
-$Comp
 L K_Resistors:10k_1206_1% R10
 U 1 1 5CC73B58
@@
 F 5 "1206S4F1002T5E" H 1800 5550 50  0001 L CNN "Supplier Part Number 1"
 	1    1800 6200
-	1    0    0    -1
-$EndComp
-$Comp
-L K_Power:+2V2 #PWR0129
-U 1 1 5CC73B60
-P 1800 6050
-F 0 "#PWR0129" H 2050 6200 50  0001 C CNN
-F 1 "+2V2" H 1805 6223 50  0000 C CNN
-F 2 "" H 1600 6350 50  0001 C CNN
-F 3 "" H 1600 6350 50  0001 C CNN
-	1    1800 6050
 	1    0    0    -1
 $EndComp
@@
 Wire Wire Line
 	3600 4450 3950 4450
-$Comp
-L K_Power:+2V2 #PWR0102
-U 1 1 5CC2A21A
-P 5950 4350
-F 0 "#PWR0102" H 6200 4500 50  0001 C CNN
-F 1 "+2V2" H 5955 4523 50  0000 C CNN
-F 2 "" H 5750 4650 50  0001 C CNN
-F 3 "" H 5750 4650 50  0001 C CNN
-	1    5950 4350
-	1    0    0    -1
-$EndComp
 Wire Wire Line
 	9150 4400 9150 5700
@@
 	7950 4400 7950 4900
 $Comp
-L K_Power:+2V2 #PWR06
-U 1 1 5CC78812
-P 9750 4600
-F 0 "#PWR06" H 10000 4750 50  0001 C CNN
-F 1 "+2V2" H 9755 4773 50  0000 C CNN
-F 2 "" H 9550 4900 50  0001 C CNN
-F 3 "" H 9550 4900 50  0001 C CNN
-	1    9750 4600
-	1    0    0    -1
-$EndComp
-$Comp
 L power:GND #PWR07
 U 1 1 5CC78BBD
@@
 $EndComp
 $Comp
-L K_Power:+2V2 #PWR08
-U 1 1 5CC7CE23
-P 10150 4600
-F 0 "#PWR08" H 10400 4750 50  0001 C CNN
-F 1 "+2V2" H 10155 4773 50  0000 C CNN
-F 2 "" H 9950 4900 50  0001 C CNN
-F 3 "" H 9950 4900 50  0001 C CNN
-	1    10150 4600
-	1    0    0    -1
-$EndComp
-$Comp
-L K_Power:+2V2 #PWR010
-U 1 1 5CC7D205
-P 10600 4600
-F 0 "#PWR010" H 10850 4750 50  0001 C CNN
-F 1 "+2V2" H 10605 4773 50  0000 C CNN
-F 2 "" H 10400 4900 50  0001 C CNN
-F 3 "" H 10400 4900 50  0001 C CNN
-	1    10600 4600
-	1    0    0    -1
-$EndComp
-$Comp
 L power:GND #PWR09
 U 1 1 5CC7D3FD
@@
 	1    0    0    -1
 $EndComp
+$Comp
+L K_Power:+2V5 #PWR0128
+U 1 1 5CC71A0D
+P 1800 6800
+F 0 "#PWR0128" H 2050 6950 50  0001 C CNN
+F 1 "+2V5" H 1805 6973 50  0000 C CNN
+F 2 "" H 1600 7100 50  0001 C CNN
+F 3 "" H 1600 7100 50  0001 C CNN
+	1    1800 6800
+	1    0    0    -1
+$EndComp
+$Comp
+L K_Power:+2V5 #PWR0129
+U 1 1 5CC73B60
+P 1800 6050
+F 0 "#PWR0129" H 2050 6200 50  0001 C CNN
+F 1 "+2V5" H 1805 6223 50  0000 C CNN
+F 2 "" H 1600 6350 50  0001 C CNN
+F 3 "" H 1600 6350 50  0001 C CNN
+	1    1800 6050
+	1    0    0    -1
+$EndComp
+$Comp
+L K_Power:+2V5 #PWR0127
+U 1 1 5CC6DEB7
+P 1800 5300
+F 0 "#PWR0127" H 2050 5450 50  0001 C CNN
+F 1 "+2V5" H 1805 5473 50  0000 C CNN
+F 2 "" H 1600 5600 50  0001 C CNN
+F 3 "" H 1600 5600 50  0001 C CNN
+	1    1800 5300
+	1    0    0    -1
+$EndComp
+$Comp
+L K_Power:+2V5 #PWR0126
+U 1 1 5CC6C3A2
+P 1800 4550
+F 0 "#PWR0126" H 2050 4700 50  0001 C CNN
+F 1 "+2V5" H 1805 4723 50  0000 C CNN
+F 2 "" H 1600 4850 50  0001 C CNN
+F 3 "" H 1600 4850 50  0001 C CNN
+	1    1800 4550
+	1    0    0    -1
+$EndComp
+$Comp
+L K_Power:+2V5 #PWR0125
+U 1 1 5CC6ACCE
+P 1800 3800
+F 0 "#PWR0125" H 2050 3950 50  0001 C CNN
+F 1 "+2V5" H 1805 3973 50  0000 C CNN
+F 2 "" H 1600 4100 50  0001 C CNN
+F 3 "" H 1600 4100 50  0001 C CNN
+	1    1800 3800
+	1    0    0    -1
+$EndComp
+$Comp
+L K_Power:+2V5 #PWR0124
+U 1 1 5CC69306
+P 1800 3050
+F 0 "#PWR0124" H 2050 3200 50  0001 C CNN
+F 1 "+2V5" H 1805 3223 50  0000 C CNN
+F 2 "" H 1600 3350 50  0001 C CNN
+F 3 "" H 1600 3350 50  0001 C CNN
+	1    1800 3050
+	1    0    0    -1
+$EndComp
+$Comp
+L K_Power:+2V5 #PWR0115
+U 1 1 5CC6330B
+P 2250 1550
+F 0 "#PWR0115" H 2500 1700 50  0001 C CNN
+F 1 "+2V5" H 2255 1723 50  0000 C CNN
+F 2 "" H 2050 1850 50  0001 C CNN
+F 3 "" H 2050 1850 50  0001 C CNN
+	1    2250 1550
+	1    0    0    -1
+$EndComp
+$Comp
+L K_Power:+2V5 #PWR0116
+U 1 1 5CC63D9D
+P 3400 900
+F 0 "#PWR0116" H 3650 1050 50  0001 C CNN
+F 1 "+2V5" H 3405 1073 50  0000 C CNN
+F 2 "" H 3200 1200 50  0001 C CNN
+F 3 "" H 3200 1200 50  0001 C CNN
+	1    3400 900
+	1    0    0    -1
+$EndComp
+$Comp
+L K_Power:+2V5 #PWR0117
+U 1 1 5CC642B6
+P 4550 1550
+F 0 "#PWR0117" H 4800 1700 50  0001 C CNN
+F 1 "+2V5" H 4555 1723 50  0000 C CNN
+F 2 "" H 4350 1850 50  0001 C CNN
+F 3 "" H 4350 1850 50  0001 C CNN
+	1    4550 1550
+	1    0    0    -1
+$EndComp
+$Comp
+L K_Power:+2V5 #PWR010
+U 1 1 5CC7D205
+P 10600 4600
+F 0 "#PWR010" H 10850 4750 50  0001 C CNN
+F 1 "+2V5" H 10605 4773 50  0000 C CNN
+F 2 "" H 10400 4900 50  0001 C CNN
+F 3 "" H 10400 4900 50  0001 C CNN
+	1    10600 4600
+	1    0    0    -1
+$EndComp
+$Comp
+L K_Power:+2V5 #PWR08
+U 1 1 5CC7CE23
+P 10150 4600
+F 0 "#PWR08" H 10400 4750 50  0001 C CNN
+F 1 "+2V5" H 10155 4773 50  0000 C CNN
+F 2 "" H 9950 4900 50  0001 C CNN
+F 3 "" H 9950 4900 50  0001 C CNN
+	1    10150 4600
+	1    0    0    -1
+$EndComp
+$Comp
+L K_Power:+2V5 #PWR06
+U 1 1 5CC78812
+P 9750 4600
+F 0 "#PWR06" H 10000 4750 50  0001 C CNN
+F 1 "+2V5" H 9755 4773 50  0000 C CNN
+F 2 "" H 9550 4900 50  0001 C CNN
+F 3 "" H 9550 4900 50  0001 C CNN
+	1    9750 4600
+	1    0    0    -1
+$EndComp
+$Comp
+L K_Power:+2V5 #PWR0108
+U 1 1 5CC3F27E
+P 9300 5350
+F 0 "#PWR0108" H 9550 5500 50  0001 C CNN
+F 1 "+2V5" H 9305 5523 50  0000 C CNN
+F 2 "" H 9100 5650 50  0001 C CNN
+F 3 "" H 9100 5650 50  0001 C CNN
+	1    9300 5350
+	1    0    0    -1
+$EndComp
+$Comp
+L K_Power:+2V5 #PWR0103
+U 1 1 5CC2A9EF
+P 8300 5700
+F 0 "#PWR0103" H 8550 5850 50  0001 C CNN
+F 1 "+2V5" H 8305 5873 50  0000 C CNN
+F 2 "" H 8100 6000 50  0001 C CNN
+F 3 "" H 8100 6000 50  0001 C CNN
+	1    8300 5700
+	1    0    0    -1
+$EndComp
+$Comp
+L K_Power:+2V5 #PWR0102
+U 1 1 5D590506
+P 5950 4350
+F 0 "#PWR0102" H 6200 4500 50  0001 C CNN
+F 1 "+2V5" H 5955 4523 50  0000 C CNN
+F 2 "" H 5750 4650 50  0001 C CNN
+F 3 "" H 5750 4650 50  0001 C CNN
+	1    5950 4350
+	1    0    0    -1
+$EndComp
